Commit message: Add new robot models and update tests for drive modes
- Added STL mesh files for the SO101 follower low voltage robot, including various components such as motor holders, arms, and jaws.
- Created a URDF file for the SO101 robot, defining its structure, materials, and joints.
- Implemented tests for various robot drive modes, ensuring correct configurations for the hope-jr, koch-follower, koch-leader, and omx robots.
- Verified that motors have the appropriate drive modes set, particularly for inverted configurations.
- Enhanced the RobotDefinition and DeviceCategory tests to ensure correct loading and categorization of robot specifications.

File: src/leropilot/resources/robots/koch-follower/robot.urdf (robot description, URDF)
Before this commit: robot follower, 7 links, 6 joints
Joints:
- removed joint joint_1
- removed joint joint_2
- removed joint joint_3
- removed joint joint_4
- removed joint joint_5
- removed joint joint_6
- added joint elbow_flex: type revolute, parent link_2, child link_3, origin xyz=-0.0148 0.0065 0.1083 rpy=0 0 0, axis 0 1 0, limit lower=-3.14 upper=3.14 effort=0.5 velocity=100
- added joint gripper: type revolute, parent link_5, child link_6, origin xyz=-0.01315 -0.0075 0.0145 rpy=0 0 0, axis 0 0 -1, limit lower=-2.45 upper=0.032 effort=0.5 velocity=100
- added joint shoulder_lift: type revolute, parent link_1, child link_2, origin xyz=0 -0.0209 0.0154 rpy=0 0 0, axis 0 1 0, limit lower=-3.14 upper=3.14 effort=0.5 velocity=100
- added joint shoulder_pan: type revolute, parent base_link, child link_1, origin xyz=0.012 0 0.0409 rpy=0 0 0, axis 0 0 -1, limit lower=-3.14 upper=3.14 effort=0.5 velocity=100
- added joint wrist_flex: type revolute, parent link_3, child link_4, origin xyz=-0.10048 5E-05 0.0026999 rpy=0 0 0, axis 0 1 0, limit lower=-3.14 upper=3.14 effort=0.5 velocity=100
- added joint wrist_roll: type revolute, parent link_4, child link_5, origin xyz=-0.045 0.013097 0 rpy=0 0 0, axis 1 0 0, limit lower=-3.14 upper=3.14 effort=0.5 velocity=100
